File: hardware/breakout_slime/breakout_slime.kicad_pcb (KiCad board)
At the start: 2 copper layers, 54.6 x 35.6 mm, 11 parts, among them J1 IMU_Conn_Female, SW1 SW_SPDT, U1 TP4056_Breakout, U2 WeMos_D1_mini, U3 BNO/MPU_Break

Commit message: Fixed battery connector polarity on breakout_slime
Parts:
- J1: renamed from BT1; value Battery_Cell -> Battery_Connector
- U3: footprint slimevr_pcb:BNO_MPU_Breakout -> slimevr_pcb:BNO_MPU_ICM_Breakout
- moved R1 0.15 mm to (76.7, 57.3)
- renumbered J1 to J2
Connections:
- J1 pad 1: /B+ -> Net-(J1-Pad1)
- J1 pad 2: Net-(BT1-Pad2) -> /B+
- U1 pad 4: Net-(BT1-Pad2) -> Net-(J1-Pad1)
- U3 pad 6: /INT1 -> unconnected-(U3-Pad6)
Routing:
- net Net-(BT1-Pad2): track 33.4 -> 0.00 mm
- net Net-(J1-Pad1): track 0.00 -> 30.6 mm
- net /B+: track 38.6 -> 41.1 mm
- net /INT1: track 70.8 -> 69.7 mm

Commit message: Filled in ground planes, updated version number, added Changelog
Routing:
- net GND: track 21.7 -> 61.8 mm, vias 2 -> 26
- net Net-(J1-Pad1): track 30.6 -> 31.5 mm
Other:
- board text added: "breakout_slime v0.1.1 by TheButlah License: CERN-OHL-P v2 or later github.com/TheButlah/slimevr_pcb"
- board text removed: "License: CERN-OHL-P v2 or later github.com/TheButlah/slimevr_pcb"
Changed lines of the file:
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@@
   (title_block
     (title "breakout_slime")
-    (date "2022-03-07")
+    (date "2022-03-10")
     (rev "0.1.1")
     (company "https://github.com/TheButlah/slimevr_pcb")
@@
   )
   (gr_rect (start 103.48652 28.81052) (end 48.87652 64.37052) (layer "Edge.Cuts") (width 0.1) (fill none))
-  (gr_text "License: CERN-OHL-P v2 or later\ngithub.com/TheButlah/slimevr_pcb\n" (at 92.05652 33.38252) (layer "B.SilkS")
-    (effects (font (size 0.8 0.8) (thickness 0.125)) (justify mirror))
+  (gr_text "breakout_slime v0.1.1 by TheButlah\nLicense: CERN-OHL-P v2 or later\ngithub.com/TheButlah/slimevr_pcb\n" (at 59.5376 31.1912) (layer "B.SilkS")
+    (effects (font (size 0.75 0.75) (thickness 0.125)) (justify mirror))
   )
   (segment (start 78.84852 39.47852) (end 76.05452 39.47852) (width 0.25) (layer "B.Cu") (net 1))
@@
   (segment (start 80.88052 39.47852) (end 93.98 52.578) (width 0.25) (layer "B.Cu") (net 1))
   (segment (start 76.05452 39.47852) (end 75.80052 39.73252) (width 0.25) (layer "B.Cu") (net 1))
-  (segment (start 95.59652 59.02052) (end 95.95652 59.02052) (width 0.25) (layer "B.Cu") (net 1))
   (segment (start 75.80052 39.73252) (end 75.80052 46.08252) (width 0.25) (layer "B.Cu") (net 1))
   (segment (start 89.77052 56.75052) (end 89.77052 58.02052) (width 0.25) (layer "B.Cu") (net 2))
@@
   (segment (start 67.16452 60.14252) (end 65.29652 58.27452) (width 0.25) (layer "F.Cu") (net 7))
   (segment (start 61.06852 58.27452) (end 65.29652 58.27452) (width 0.25) (layer "F.Cu") (net 7))
+  (segment (start 94.0308 50.546) (end 93.0656 50.546) (width 0.5) (layer "F.Cu") (net 8))
+  (segment (start 77.5716 54.6608) (end 79.756 54.6608) (width 0.5) (layer "F.Cu") (net 8))
+  (segment (start 86.6648 46.6852) (end 86.6648 46.736) (width 0.5) (layer "F.Cu") (net 8))
+  (segment (start 56.4896 57.3024) (end 56.4896 54.7624) (width 0.5) (layer "F.Cu") (net 8))
   (segment (start 84.016031 57.933009) (end 81.13452 60.81452) (width 0.5) (layer "F.Cu") (net 8))
+  (segment (start 84.836 51.308) (end 86.7156 53.1876) (width 0.5) (layer "F.Cu") (net 8))
   (segment (start 81.13452 60.81452) (end 80.88052 60.81452) (width 0.5) (layer "F.Cu") (net 8))
+  (segment (start 95.4024 49.1744) (end 94.0308 50.546) (width 0.5) (layer "F.Cu") (net 8))
+  (segment (start 66.9544 51.308) (end 66.9544 50.1904) (width 0.5) (layer "F.Cu") (net 8))
+  (segment (start 65.532 48.768) (end 67.7672 46.5328) (width 0.5) (layer "F.Cu") (net 8))
+  (segment (start 93.0656 50.546) (end 91.5416 52.07) (width 0.5) (layer "F.Cu") (net 8))
+  (segment (start 67.7672 46.5328) (end 67.7672 46.1772) (width 0.5) (layer "F.Cu") (net 8))
+  (segment (start 83.9724 40.6908) (end 83.9724 40.9956) (width 0.5) (layer "F.Cu") (net 8))
+  (segment (start 83.9724 40.9956) (end 82.296 42.672) (width 0.5) (layer "F.Cu") (net 8))
+  (segment (start 88.646 44.9072) (end 90.5256 43.0276) (width 0.5) (layer "F.Cu") (net 8))
+  (segment (start 96.3676 49.1744) (end 95.4024 49.1744) (width 0.5) (layer "F.Cu") (net 8))
+  (segment (start 88.4428 44.9072) (end 86.6648 46.6852) (width 0.5) (layer "F.Cu") (net 8))
   (segment (start 78.525911 50.65452) (end 84.016031 56.14464) (width 0.5) (layer "F.Cu") (net 8))
+  (segment (start 84.328 51.308) (end 84.836 51.308) (width 0.5) (layer "F.Cu") (net 8))
+  (segment (start 88.4428 44.9072) (end 88.646 44.9072) (width 0.5) (layer "F.Cu") (net 8))
+  (segment (start 79.756 54.6608) (end 80.01 54.4068) (width 0.5) (layer "F.Cu") (net 8))
+  (segment (start 54.5084 57.15) (end 54.5084 54.8132) (width 0.5) (layer "F.Cu") (net 8))
   (segment (start 77.07052 50.65452) (end 78.525911 50.65452) (width 0.5) (layer "F.Cu") (net 8))
+  (segment (start 83.9724 40.6908) (end 85.9028 38.7604) (width 0.5) (layer "F.Cu") (net 8))
+  (segment (start 89.8652 60.6044) (end 89.4588 60.198) (width 0.5) (layer "F.Cu") (net 8))
+  (segment (start 59.1312 41.9608) (end 58.7756 42.3164) (width 0.5) (layer "F.Cu") (net 8))
+  (segment (start 66.9544 50.1904) (end 65.532 48.768) (width 0.5) (layer "F.Cu") (net 8))
   (segment (start 84.016031 56.14464) (end 84.016031 57.933009) (width 0.5) (layer "F.Cu") (net 8))
+  (segment (start 92.202 60.6044) (end 89.8652 60.6044) (width 0.5) (layer "F.Cu") (net 8))
+  (segment (start 54.5084 54.8132) (end 54.5592 54.7624) (width 0.5) (layer "F.Cu") (net 8))
+  (segment (start 59.1312 39.4716) (end 59.1312 41.9608) (width 0.5) (layer "F.Cu") (net 8))
+  (segment (start 56.4896 54.7624) (end 56.5404 54.7116) (width 0.5) (layer "F.Cu") (net 8))
+  (via (at 96.3676 49.1744) (size 0.8) (drill 0.4) (layers "F.Cu" "B.Cu") (free) (net 8))
+  (via (at 56.4896 57.3024) (size 0.8) (drill 0.4) (layers "F.Cu" "B.Cu") (free) (net 8))
+  (via (at 88.4428 44.9072) (size 0.8) (drill 0.4) (layers "F.Cu" "B.Cu") (free) (net 8))
+  (via (at 89.4588 60.198) (size 0.8) (drill 0.4) (layers "F.Cu" "B.Cu") (net 8))
+  (via (at 80.01 54.4068) (size 0.8) (drill 0.4) (layers "F.Cu" "B.Cu") (free) (net 8))
+  (via (at 84.328 51.308) (size 0.8) (drill 0.4) (layers "F.Cu" "B.Cu") (free) (net 8))
   (via (at 80.88052 60.81452) (size 0.8) (drill 0.4) (layers "F.Cu" "B.Cu") (free) (net 8))
+  (via (at 82.296 42.672) (size 0.8) (drill 0.4) (layers "F.Cu" "B.Cu") (free) (net 8))
   (via (at 77.07052 50.65452) (size 0.8) (drill 0.4) (layers "F.Cu" "B.Cu") (free) (net 8))
+  (via (at 67.7672 46.1772) (size 0.8) (drill 0.4) (layers "F.Cu" "B.Cu") (net 8))
+  (via (at 77.5716 54.6608) (size 0.8) (drill 0.4) (layers "F.Cu" "B.Cu") (free) (net 8))
+  (via (at 56.5404 54.7116) (size 0.8) (drill 0.4) (layers "F.Cu" "B.Cu") (net 8))
+  (via (at 83.9724 40.6908) (size 0.8) (drill 0.4) (layers "F.Cu" "B.Cu") (free) (net 8))
+  (via (at 92.202 60.6044) (size 0.8) (drill 0.4) (layers "F.Cu" "B.Cu") (free) (net 8))
+  (via (at 54.5592 54.7624) (size 0.8) (drill 0.4) (layers "F.Cu" "B.Cu") (net 8))
+  (via (at 85.9028 38.7604) (size 0.8) (drill 0.4) (layers "F.Cu" "B.Cu") (net 8))
+  (via (at 65.532 48.768) (size 0.8) (drill 0.4) (layers "F.Cu" "B.Cu") (net 8))
+  (via (at 58.7756 42.3164) (size 0.8) (drill 0.4) (layers "F.Cu" "B.Cu") (free) (net 8))
+  (via (at 90.5256 43.0276) (size 0.8) (drill 0.4) (layers "F.Cu" "B.Cu") (free) (net 8))
+  (via (at 59.1312 39.4716) (size 0.8) (drill 0.4) (layers "F.Cu" "B.Cu") (free) (net 8))
+  (via (at 66.9544 51.308) (size 0.8) (drill 0.4) (layers "F.Cu" "B.Cu") (free) (net 8))
+  (via (at 54.5084 57.15) (size 0.8) (drill 0.4) (layers "F.Cu" "B.Cu") (free) (net 8))
+  (via (at 91.5416 52.07) (size 0.8) (drill 0.4) (layers "F.Cu" "B.Cu") (free) (net 8))
+  (via (at 86.7156 53.1876) (size 0.8) (drill 0.4) (layers "F.Cu" "B.Cu") (free) (net 8))
+  (via (at 94.0308 50.546) (size 0.8) (drill 0.4) (layers "F.Cu" "B.Cu") (free) (net 8))
+  (via (at 86.6648 46.736) (size 0.8) (drill 0.4) (layers "F.Cu" "B.Cu") (net 8))
   (segment (start 65.16452 57.84652) (end 68.03852 54.97252) (width 0.5) (layer "B.Cu") (net 8))
   (segment (start 65.16452 60.14252) (end 65.16452 57.84652) (width 0.5) (layer "B.Cu") (net 8))
@@
   (segment (start 76.81652 57.25852) (end 76.81652 52.68652) (width 0.25) (layer "F.Cu") (net 12))
   (via (at 76.81652 52.68652) (size 0.8) (drill 0.4) (layers "F.Cu" "B.Cu") (net 12))
-  (segment (start 71.84504 52.03304) (end 60.56052 40.74852) (width 0.25) (layer "B.Cu") (net 12))
-  (segment (start 76.16304 52.03304) (end 71.84504 52.03304) (width 0.25) (layer "B.Cu") (net 12))
+  (segment (start 71.9836 52.1716) (end 60.56052 40.74852) (width 0.25) (layer "B.Cu") (net 12))
+  (segment (start 76.3016 52.1716) (end 71.9836 52.1716) (width 0.25) (layer "B.Cu") (net 12))
   (segment (start 60.56052 40.74852) (end 50.63152 40.74852) (width 0.25) (layer "B.Cu") (net 12))
-  (segment (start 76.81652 52.68652) (end 76.16304 52.03304) (width 0.25) (layer "B.Cu") (net 12))
+  (segment (start 76.81652 52.68652) (end 76.3016 52.1716) (width 0.25) (layer "B.Cu") (net 12))
   (segment (start 52.75052 60.81452) (end 52.75052 51.22652) (width 0.25) (layer "F.Cu") (net 13))
   (segment (start 76.56252 35.92252) (end 75.40104 37.084) (width 0.25) (layer "F.Cu") (net 13))
@@
   (via (at 52.75052 43.617209) (size 0.8) (drill 0.4) (layers "F.Cu" "B.Cu") (net 13))
   (segment (start 52.75052 51.22652) (end 52.75052 43.617209) (width 0.25) (layer "B.Cu") (net 13))
-  (segment (start 95.95652 50.49052) (end 95.95652 57.02052) (width 0.25) (layer "B.Cu") (net 24))
-  (segment (start 78.781026 33.74859) (end 79.21459 33.74859) (width 0.25) (layer "B.Cu") (net 24))
-  (segment (start 79.21459 33.74859) (end 95.95652 50.49052) (width 0.25) (layer "B.Cu") (net 24))
+  (segment (start 97.4852 55.49184) (end 95.95652 57.02052) (width 0.25) (layer "B.Cu") (net 24))
+  (segment (start 79.21459 33.74859) (end 97.4852 52.0192) (width 0.25) (layer "B.Cu") (net 24))
+  (segment (start 97.4852 52.0192) (end 97.4852 55.49184) (width 0.25) (layer "B.Cu") (net 24))
   (zone (net 8) (net_name "GND") (layer "B.Cu") (hatch edge 0.508)
     (priority 1)

Commit message: breakout_slime v0.1.2
Parts:
- moved J1 0.61 mm to (96.3, 57.5)
Connections:
- net /5V renamed +5V
- net /B+ renamed B+
- net /INT1 renamed INT1
- net /INT2 renamed INT2
- net /SCL renamed SCL
- net /SDA renamed SDA
Routing:
- net GND: track 61.8 -> 11.4 mm, vias 26 -> 49
- net B+: track 40.8 -> 41.6 mm
- added copper zone on F.Cu, net GND
Other:
- outline, holes or cut-outs redrawn
- board text added: "${REVISION}"
