File: hardware/breakout_slime/breakout_slime.kicad_pcb (KiCad board)
At the start: 2 copper layers, 54.6 x 35.3 mm, 11 parts, among them J1 Battery_Connector, J2 IMU_Conn_Female, SW1 SW_SPDT, U1 TP4056_Breakout, U2 WeMos_D1_mini, U3 BNO/MPU_Break

Commit message: [breakout_slime] Released v0.1.4
Parts:
- moved D1 4.59 mm to (89.8, 60.1)
- moved J2 4.15 mm to (75.3, 60.3)
- moved SW1 0.18 mm to (56.6, 60.8)
Routing:
- net Net-(JP1-Pad1): track 33.8 -> 23.8 mm
- net SDA: track 40.5 -> 48.9 mm
- net SCL: track 44.3 -> 40.0 mm, vias 0 -> 1
- net INT2: track 24.8 -> 28.7 mm
- net +5V: track 18.1 -> 21.9 mm
- net Net-(D1-Pad2): track 34.0 -> 30.5 mm
- net +3V3: track 45.7 -> 42.9 mm
- net GND: track 11.6 -> 10.7 mm, vias 52 -> 53
