File: hardware/breakout_slime/breakout_slime.kicad_sch (KiCad schematic)
At the start: 11 parts, among them J1 Battery_Connector, J2 IMU_Conn_Female, SW1 SW_SPDT, U1 TP4056_Breakout, U2 WeMos_D1_mini, U3 BNO/MPU_Break

Commit message: breakout_slime v0.1.2
Connections:
- net 5V renamed +5V
Other:
- moved on the sheet: U3

Commit message: [breakout_slime] Released v0.1.3
Connections:
- net B+: now also J1.1 (Pin_1); no longer J1.2 (Pin_2)
- net at U1.4 (B-): now also J1.2 (Pin_2); no longer J1.1 (Pin_1)
Changed lines of the file:
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@@
   (title_block
     (title "breakout_slime")
-    (date "2022-03-12")
-    (rev "0.1.2")
+    (date "2022-04-13")
+    (rev "0.1.3")
     (company "https://github.com/TheButlah/slimevr_pcb")
     (comment 1 "Licensed under CERN-OHL-P v2 or later")
@@
     (stroke (width 0) (type default) (color 0 0 0 0))
   )
+  (wire (pts (xy 73.66 53.34) (xy 73.66 55.88))
+    (stroke (width 0) (type default) (color 0 0 0 0))
+  )
   (wire (pts (xy 73.66 50.8) (xy 73.66 53.34))
     (stroke (width 0) (type default) (color 0 0 0 0))
@@
     (stroke (width 0) (type default) (color 0 0 0 0))
   )
+  (wire (pts (xy 73.66 58.42) (xy 73.66 60.96))
+    (stroke (width 0) (type default) (color 0 0 0 0))
+  )
   (wire (pts (xy 36.83 26.67) (xy 36.83 49.53))
     (stroke (width 0) (type default) (color 0 0 0 0))
@@
     (stroke (width 0) (type default) (color 0 0 0 0))
   )
-  (wire (pts (xy 73.66 53.34) (xy 73.66 55.88))
-    (stroke (width 0) (type default) (color 0 0 0 0))
-  )
   (polyline (pts (xy 13.97 13.97) (xy 13.97 95.25))
     (stroke (width 0) (type default) (color 0 0 0 0))
   )
-  (wire (pts (xy 73.66 58.42) (xy 73.66 60.96))
-    (stroke (width 0) (type default) (color 0 0 0 0))
-  )
   (wire (pts (xy 69.85 26.67) (xy 36.83 26.67))
     (stroke (width 0) (type default) (color 0 0 0 0))
@@
     (stroke (width 0) (type default) (color 0 0 0 0))
   )
+  (wire (pts (xy 69.85 69.85) (xy 69.85 64.77))
+    (stroke (width 0) (type default) (color 0 0 0 0))
+  )
+  (wire (pts (xy 172.72 31.75) (xy 179.07 31.75))
+    (stroke (width 0) (type default) (color 0 0 0 0))
+  )
+  (wire (pts (xy 184.15 60.96) (xy 182.88 60.96))
+    (stroke (width 0) (type default) (color 0 0 0 0))
+  )
+  (wire (pts (xy 182.88 76.2) (xy 182.88 80.01))
+    (stroke (width 0) (type default) (color 0 0 0 0))
+  )
   (wire (pts (xy 67.31 60.96) (xy 73.66 60.96))
-    (stroke (width 0) (type default) (color 0 0 0 0))
-  )
-  (wire (pts (xy 69.85 69.85) (xy 69.85 64.77))
-    (stroke (width 0) (type default) (color 0 0 0 0))
-  )
-  (wire (pts (xy 172.72 31.75) (xy 179.07 31.75))
-    (stroke (width 0) (type default) (color 0 0 0 0))
-  )
-  (wire (pts (xy 184.15 60.96) (xy 182.88 60.96))
-    (stroke (width 0) (type default) (color 0 0 0 0))
-  )
-  (wire (pts (xy 182.88 76.2) (xy 182.88 80.01))
     (stroke (width 0) (type default) (color 0 0 0 0))
   )
@@
     (pin "2")
   )
-  (symbol (lib_id "Connector:Conn_01x02_Female") (at 78.74 58.42 0) (mirror x) (unit 1)
+  (symbol (lib_id "Connector:Conn_01x02_Female") (at 78.74 55.88 0) (unit 1)
     (in_bom yes) (on_board yes)
-    (property "Reference" "J1" (id 0) (at 78.105 50.8 0))
-    (property "Value" "Battery_Connector" (id 1) (at 85.09 53.34 0))
-    (property "Footprint" "Connector_JST:JST_PH_S2B-PH-K_1x02_P2.00mm_Horizontal" (id 2) (at 78.74 58.42 0)
-      (effects (font (size 1.27 1.27)) hide)
-    )
-    (property "Datasheet" "~" (id 3) (at 78.74 58.42 0)
-      (effects (font (size 1.27 1.27)) hide)
-    )
+    (property "Reference" "J1" (id 0) (at 78.74 53.34 0))
+    (property "Value" "Battery_Connector" (id 1) (at 83.82 60.96 0))
+    (property "Footprint" "Connector_JST:JST_PH_S2B-PH-K_1x02_P2.00mm_Horizontal" (id 2) (at 78.74 55.88 0)
+      (effects (font (size 1.27 1.27)) hide)
+    )
+    (property "Datasheet" "~" (id 3) (at 78.74 55.88 0)
+      (effects (font (size 1.27 1.27)) hide)
+    )
