File: hardware/ferrous_slime/ferrous_slime.kicad_pcb (KiCad board)
At the start: 2 copper layers, 41.4 x 34.1 mm, 54 parts, among them J1 IMU_Connector, J2 Unused_IO, J3 Battery_Connector, J4 USB_C_Receptacle_USB2.0, Q1 DMG3415U, SW1 SW_PWR, U1 BNO/MPU/ICM_Break, U2 ESP32-C3-MINI-1, U3 TP4056, U4 M3406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

Commit message: Added refs to silkscreen
Parts:
- D5: value LED -> LED_PROG
- Q1: value DMG3415U -> CJ2305
- moved C5 0.82 mm to (59.4, 57.5), turned to -90 degrees
Routing:
- net GND: vias 111 -> 112

Commit message: v0.1.0 board released
Parts:
- added G***: LOGO, slimevr_pcb:oshw_cert, B.Cu at (94.3, 35.9)
- added G***: LOGO, slimevr_pcb:oshw_logo, B.Cu at (59.2, 60.7)
- D1: footprint Diode_SMD:D_SOD-323_HandSoldering -> slimevr_pcb:SOD882
- D5: value LED_PROG -> LED
- L1: footprint Inductor_SMD:L_7.3x7.3_H4.5 -> Inductor_SMD:L_Wuerth_MAPI-3015
- R4: value 100kR 1% -> 120K
- moved L1 0.89 mm to (85.0, 57.3)
- moved D1 0.75 mm to (69.8, 50.0)
- moved U4 0.10 mm to (89.7, 58.2)
Routing:
- net +3V3: track 123.1 -> 125.3 mm, vias 8 -> 7
- net GND: track 45.8 -> 46.1 mm, vias 112 -> 113
Other:
- board size 41.4 x 34.1 mm -> 41.4 x 34 mm
- board text added: "For use with SlimeVR Made with <3"

Commit message: Finished pcb for ferrous_slime v0.2.0
Parts:
- added H1: MountingHole_2.1mm, MountingHole:MountingHole_2.1mm, F.Cu at (64.8, 60.8)
- added H2: MountingHole_2.1mm, MountingHole:MountingHole_2.1mm, F.Cu at (85.6, 59.6)
- added H3: MountingHole_2.1mm, MountingHole:MountingHole_2.1mm, F.Cu at (61.7, 32.3)
- added JP4: VCC_GBIM, Jumper:SolderJumper-2_P1.3mm_Open_RoundedPad1.0x1.5mm, B.Cu at (62.6, 55.6)
- D3: value LED_CHRG -> CHRG
- D4: value LED_FULL -> FULL
- D5: value LED -> LED_IO5
- G***: moved to F.Cu
- JP1: value ICM/MPU_AD0 -> +AD0_GI/GM; moved to B.Cu
- JP2: value INT_ICM/ADO_BNO -> INT_ABGI/-ADO_GB; moved to B.Cu
- JP3: value BNO/MPU_INT1 -> INT_GB/GM; moved to B.Cu
- U1: footprint slimevr_pcb:BNO_MPU_ICM_Breakout -> slimevr_pcb:AB_GB_GM_GI_Breakout
- moved C5 9.80 mm to (68.8, 54.7)
- moved JP3 6.58 mm to (58.2, 60.3), turned to -90 degrees
- moved JP1 5.95 mm to (59.6, 55.5), turned to -90 degrees
- moved L1 2.74 mm to (86.0, 54.7)
- moved JP2 2.72 mm to (61.7, 60.5), turned to 90 degrees
- moved G*** 0.65 mm to (58.5, 60.6), turned to 0 degrees
- moved D1 0.64 mm to (70.5, 50.0)
- moved C4 0.56 mm to (68.1, 48.6)
- moved J1 0.44 mm to (69.8, 58.4)
- moved U1 0.25 mm to (58.2, 43.1)
Connections:
- U1 pad 1: +3V3 -> Net-(JP4-Pad2)
Routing:
- net Net-(JP1-Pad1): track 25.3 -> 14.5 mm, vias 0 -> 1
- net +3V3: track 125.3 -> 119.1 mm
- net Net-(JP1-Pad3): track 31.3 -> 25.7 mm, vias 1 -> 0
- net IO6_INT1: track 26.2 -> 30.4 mm, vias 2 -> 3
- net Net-(JP2-Pad2): track 22.6 -> 19.0 mm, vias 2 -> 1
- net GND: track 46.1 -> 43.2 mm, vias 113 -> 109
- net Net-(JP4-Pad2): track 0.00 -> 2.27 mm
- net Net-(C2-Pad1): track 33.1 -> 31.5 mm
- net Net-(JP3-Pad3): track 28.8 -> 30.1 mm
- net Net-(L1-Pad1): track 6.82 -> 8.03 mm
- net IO8_SCL: track 36.6 -> 37.7 mm
- net IO7_INT2: track 21.7 -> 20.7 mm
- net UNUSED_IO9: track 30.9 -> 31.6 mm
- net UNUSED_IO21: track 48.4 -> 49.1 mm
Other:
- outline, holes or cut-outs redrawn

Commit message: ferrous_slime: v0.3.0
Parts:
- U1: value BNO/MPU/ICM_Break -> IMU_Breakout; footprint slimevr_pcb:AB_GB_GM_GI_Breakout -> slimevr_pcb:IMU_Breakout
- moved G*** 0.13 mm to (58.5, 60.5)
- moved J3 0.11 mm to (89.0, 49.4)
- moved D8 0.07 mm to (92.2, 43.6)
- renumbered C8 to C7, C7 to C8, R3 to R2, R2 to R3
Connections:
- J3 pad 1: GND -> +BATT
- J3 pad 2: +BATT -> GND
- R3 pad 2: VBUS -> Net-(R3-Pad2)
- U3 pad 2: VBUS -> Net-(R3-Pad2)
- U3 pad 9: unconnected-(U3-Pad9) -> GND
Routing:
- net VBUS: track 37.2 -> 34.2 mm
- net Net-(R3-Pad2): track 0.00 -> 2.25 mm
- net Net-(J4-PadA5): track 7.23 -> 6.05 mm
- net IO8_SCL: track 37.7 -> 37.0 mm
- net GND: track 43.2 -> 42.8 mm, vias 109 -> 115
Other:
- board text removed: "B+"

Commit message: Lots of pcb progress
Parts:
- removed D7, D9: LESD5D5.0CT1G, Diode_SMD:D_SOD-523
- removed D8: B5819W, Diode_SMD:D_SOD-123
- removed the R13 at (87.1, 30.9)
- removed the R14 at (91.2, 41.6)
- added R11: 120K 1%, Resistor_SMD:R_0603_1608Metric, F.Cu at (81.5, 51.1)
- added R12: 30K 1%, Resistor_SMD:R_0603_1608Metric, F.Cu at (81.5, 52.7)
- added R15: 5k1R 1%, Resistor_SMD:R_0603_1608Metric, F.Cu at (88.9, 31.6)
- added R16: 5k1R 1%, Resistor_SMD:R_0603_1608Metric, F.Cu at (87.4, 31.6)
- added U5: SRV05-4, Package_TO_SOT_SMD:SOT-23-6, F.Cu at (87.6, 34.9)
- D6: value LESD5D5.0CT1G -> B5819W; footprint Diode_SMD:D_SOD-523 -> Diode_SMD:D_SOD-123
- R10: value 30K 1% -> 120K
- R8: value 120K -> 10K
- R9: value 120K 1% -> 10K
- TP1, TP2: moved to B.Cu
- moved R10 28.1 mm to (95.5, 41.3), turned to 0 degrees
- moved R8 25.7 mm to (68.1, 49.8), turned to -90 degrees
- moved TP1 22.4 mm to (71.9, 42.5), turned to 180 degrees
- moved C1 20.3 mm to (67.6, 35.8), turned to 180 degrees
- moved R5 15.9 mm to (95.1, 43.6)
- moved D3 15.9 mm to (93.6, 43.6), turned to -90 degrees
- moved C3 15.8 mm to (67.6, 37.3), turned to 180 degrees
- moved D2 13.7 mm to (81.9, 59.1), turned to 90 degrees
- moved R3 11.8 mm to (85.9, 31.6), turned to -90 degrees
- moved D4 11.7 mm to (92.1, 43.6)
- moved R6 11.6 mm to (90.6, 43.6)
- moved C4 9.02 mm to (68.3, 39.6)
- moved D1 8.66 mm to (68.3, 41.7), turned to 0 degrees
- moved D6 8.52 mm to (83.9, 32.5), turned to 90 degrees
- moved C7 7.10 mm to (83.5, 37.7)
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- renumbered R11 to R13, R12 to R14
Connections:
- D6 pad 1: USB_D- -> VBUS
- D6 pad 2: GND -> Net-(D6-Pad2)
- J4 pad A4: Net-(D8-Pad2) -> Net-(D6-Pad2)
- J4 pad A9: Net-(D8-Pad2) -> Net-(D6-Pad2)
- J4 pad B4: Net-(D8-Pad2) -> Net-(D6-Pad2)
- J4 pad B9: Net-(D8-Pad2) -> Net-(D6-Pad2)
- R10 pad 1: B_SENSE -> Net-(J4-PadS1)
- R8 pad 1: Net-(J4-PadS1) -> +3V3
- R8 pad 2: GND -> IO10_SDA
- R9 pad 1: +BATT -> +3V3
- R9 pad 2: B_SENSE -> IO8_SCL
Routing:
- net +BATT: track 65.8 -> 24.8 mm, vias 5 -> 3
- net GND: track 42.8 -> 18.1 mm, vias 115 -> 65
- net Net-(C2-Pad1): track 31.5 -> 7.31 mm, vias 4 -> 1
- net Net-(D6-Pad2): track 0.00 -> 22.4 mm, vias 0 -> 3
- net +3V3: track 119.1 -> 97.7 mm, vias 7 -> 2
- net Net-(R3-Pad2): track 2.25 -> 18.5 mm, vias 0 -> 2
- net Net-(D8-Pad2): track 15.9 -> 0.00 mm
- net IO0: track 19.9 -> 8.15 mm, vias 2 -> 0
- net Net-(J4-PadS1): track 30.9 -> 19.2 mm, vias 1 -> 0
- net IO1: track 17.8 -> 8.36 mm, vias 2 -> 0
- net VBUS: track 34.2 -> 43.3 mm, vias 0 -> 2
- net IO7_INT2: track 20.7 -> 14.3 mm, vias 3 -> 0
- net USB_D+: track 25.3 -> 19.1 mm
- net Net-(R5-Pad1): track 2.27 -> 8.42 mm, vias 0 -> 2
- net USB_D-: track 25.0 -> 19.7 mm
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Other:
- outline, holes or cut-outs redrawn

Commit message: tmp
Parts:
- moved ${REFERENCE} 12.4 mm to (74.8, 54.6)
- moved D6 1.27 mm to (83.9, 33.8)
- moved C6 0.25 mm to (70.4, 50.8)
- moved C8 0.25 mm to (73.4, 50.8)
- moved R2 0.25 mm to (71.9, 50.8)
- moved Y1 0.25 mm to (71.4, 48.1)
- renumbered TP1 to ${REFERENCE}
Connections:
- U5 pad 2: unconnected-(U5-Pad2) -> GND
Routing:
- net Net-(C2-Pad1): track 7.31 -> 20.6 mm
- net IO1: track 8.36 -> 3.98 mm
- net +BATT: track 24.8 -> 26.3 mm, vias 3 -> 2
- net +3V3: track 97.7 -> 96.6 mm
- net VBUS: track 43.3 -> 42.3 mm
- net Net-(D6-Pad2): track 22.4 -> 21.6 mm
- net IO0: track 8.15 -> 7.40 mm
- net Net-(D2-Pad1): track 27.7 -> 27.0 mm
- net USB_D+: track 19.1 -> 18.5 mm
- net USB_D-: track 19.7 -> 19.1 mm
- net GND: track 18.1 -> 18.3 mm, vias 65 -> 117
Other:
- outline, holes or cut-outs redrawn

Commit message: Finished work
Parts:
- TP1: renamed from ${REFERENCE}; moved to F.Cu
- TP2: moved to F.Cu
- moved TP2 11.9 mm to (81.8, 48.8), turned to -90 degrees
- moved TP1 0.90 mm to (73.9, 54.5), turned to 0 degrees
Routing:
- net +BATT: track 26.3 -> 22.9 mm
- net Net-(C2-Pad1): track 20.6 -> 21.0 mm, vias 1 -> 2
- net GND: vias 117 -> 116
Other:
- outline, holes or cut-outs redrawn
